File: Hardware/LED Strip Controller/Server Rack LED Controller.kicad_sch (KiCad schematic)
At the start: 164 parts, among them J1 Conn_01x03_Male, J10 UART, J11 CONN_2, J12 Conn_01x03_Male, J13 CONN_3, J14 Conn_01x03_Male, J15 Conn_01x06_Male, J16 CONN_4, J17 TST, J18 Conn_01x02_Female, J19 Conn_02x04_Odd_Even, J2 Screw_Terminal_01x02, J20 Conn_02x04_Odd_Even, J3 PWR_SWITCH, J4 Conn_02x03_Odd_Even, J5 Conn_01x03_Female, J6 CONN_1, J7 Conn_01x03_Male, J8 SWD, J9 USB_B_Micro, Q1 IRF510N, Q10 IRF510N, Q11 IRF510N, Q12 IRF510N, Q13 IRF510N, Q14 IRF510N, Q2 IRF510N, Q3 Q_PMOS_SDG, Q4 IRF510N, Q5 IRF510N, Q6 IRF510N, Q7 IRF510N, Q8 IRF510N, Q9 IRF510N, SW1 SW_Push_Dual, U1 STM32F103C8Tx, U2 LM2596S-5, U3 LD1117S50TR_SOT223, U4 LD39050PU33R, U5 INA169, U6 USBLC6-2SC6, Y1 Crystal, Y2 8MHz

Commit message: Adding Fuse Holder and updating Kicad Schematic with new PSU connecotors, also started doing some of the layout
Parts:
- removed J12, J14, J7: Conn_01x03_Male, Connector_PinHeader_2.54mm:PinHeader_1x03_P2.54mm_Vertical, symbol Connector:Conn_01x03_Male
- added F2, F3, F4, F5: 1A, Fuse:Fuseholder_Clip-5x20mm_Littelfuse_111_Inline_P20.00x5.00mm_D1.05mm_Horizontal, symbol Device:Fuse
- added J12: LED_THREE_PWR, Connector_PinHeader_2.54mm:PinHeader_2x03_P2.54mm_Vertical, symbol Connector_Generic:Conn_02x03_Odd_Even
- added J14: LED_FOUR_PWR, Connector_PinHeader_2.54mm:PinHeader_2x03_P2.54mm_Vertical, symbol Connector_Generic:Conn_02x03_Odd_Even
- added J21: Conn_01x02_Female, Connector_JST:JST_EH_B2B-EH-A_1x02_P2.50mm_Vertical, symbol Connector:Conn_01x02_Female
- added J7: LED_TWO_PWR, Connector_PinHeader_2.54mm:PinHeader_2x03_P2.54mm_Vertical, symbol Connector_Generic:Conn_02x03_Odd_Even
- added J?: Screw_Terminal_01x02, TerminalBlock_Phoenix:TerminalBlock_Phoenix_MKDS-1,5-2-5.08_1x02_P5.08mm_Horizontal, symbol Connector:Screw_Terminal_01x02
- added Q?: Q_PMOS_SDG, Package_TO_SOT_SMD:TO-252-3_TabPin2, symbol Device:Q_PMOS_GDS
- added R?: 10K, Resistor_SMD:R_1206_3216Metric_Pad1.30x1.75mm_HandSolder, symbol Device:R
- F1: footprint Fuse:Fuseholder_Clip-5x20mm_Eaton_1A5601-01_Inline_P20.80x6.76mm_D1.70mm_Horizontal -> Fuse:Fuseholder_Clip-5x20mm_Littelfuse_111_Inline_P20.00x5.00mm_D1.05mm_Horizontal
- J1: value Conn_01x03_Male -> LED_ONE_PWR; footprint Connector_PinHeader_2.54mm:PinHeader_1x03_P2.54mm_Vertical -> Connector_PinHeader_2.54mm:PinHeader_2x03_P2.54mm_Vertical; symbol Connector:Conn_01x03_Male -> Connector_Generic:Conn_02x03_Odd_Even
- U4: footprint SON95P300X300X100-7N -> DFN-6-1EP_3x3mm_P0.95mm_EP1.7x2.6mm
Connections:
- net CONN_1_5V: now also J1.3 (Pin_3), J1.4 (Pin_4), F2.1; no longer J1.2 (Pin_2), J6.1 (Pin_1)
- net CONN_2_5V: now also F3.1, J7.3 (Pin_3), J7.4 (Pin_4); no longer J11.1 (Pin_1)
- net CONN_3_5V: now also F4.1, J12.3 (Pin_3), J12.4 (Pin_4); no longer J13.1 (Pin_1)
- net CONN_4_5V: now also F5.1, J14.3 (Pin_3), J14.4 (Pin_4); no longer J16.1 (Pin_1)
- net EXT_5V: now also J1.5 (Pin_5), J1.6 (Pin_6), J12.5 (Pin_5), J12.6 (Pin_6), J14.5 (Pin_5), J14.6 (Pin_6), J7.5 (Pin_5), J7.6 (Pin_6), Q?.3 (S); no longer J1.3 (Pin_3)
- net GND: now also R34.2, U5.1, J21.2 (Pin_2), J?.2 (Pin_2), R?.2; no longer R34.1, U1.14 (PA4)
- net PWR_5V: now also J1.2 (Pin_2), J12.1 (Pin_1), J12.2 (Pin_2), J14.1 (Pin_1), J14.2 (Pin_2), J7.1 (Pin_1), J7.2 (Pin_2)
- net RESET: now also J21.1 (Pin_1)
- new net: F3.2, J11.1 (Pin_1)
- new net: F5.2, J16.1 (Pin_1)
- new net: Q?.1 (G), R?.1
- new net: F2.2, J6.1 (Pin_1)
- new net: F4.2, J13.1 (Pin_1)
- new net: J?.1 (Pin_1), Q?.2 (D)
- new net CURR_SENSE: R34.1, U1.14 (PA4)
Other:
- note added: "Double Connector for 6A current rating (3A Per Pin)"
- note added: "External Power Supply Connection"
- moved on the sheet: C14, D10, D11, D12, D7, D8, D9, J11, J13, J16, J6, Q5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

Commit message: Adding missing changes
Parts:
- gave numbers to parts that had none: 3
Changed lines of the file:
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@@
   (symbol (lib_id "Device:R") (at 440.69 532.13 0) (unit 1)
     (in_bom yes) (on_board yes) (fields_autoplaced)
-    (property "Reference" "R?" (id 0) (at 443.23 530.8599 0)
+    (property "Reference" "R46" (id 0) (at 443.23 530.8599 0)
       (effects (font (size 1.27 1.27)) (justify left))
     )
@@
   (symbol (lib_id "power:GND") (at 440.69 542.29 0) (unit 1)
     (in_bom yes) (on_board yes) (fields_autoplaced)
-    (property "Reference" "#PWR?" (id 0) (at 440.69 548.64 0)
+    (property "Reference" "#PWR0176" (id 0) (at 440.69 548.64 0)
       (effects (font (size 1.27 1.27)) hide)
     )
@@
   (symbol (lib_id "Connector:Screw_Terminal_01x02") (at 411.48 519.43 0) (mirror y) (unit 1)
     (in_bom yes) (on_board yes) (fields_autoplaced)
-    (property "Reference" "J?" (id 0) (at 411.48 513.08 0))
+    (property "Reference" "J22" (id 0) (at 411.48 513.08 0))
     (property "Value" "Screw_Terminal_01x02" (id 1) (at 411.48 515.62 0))
     (property "Footprint" "TerminalBlock_Phoenix:TerminalBlock_Phoenix_MKDS-1,5-2-5.08_1x02_P5.08mm_Horizontal" (id 2) (at 411.48 519.43 0)
@@
   (symbol (lib_id "Device:Q_PMOS_GDS") (at 440.69 521.97 90) (unit 1)
     (in_bom yes) (on_board yes) (fields_autoplaced)
-    (property "Reference" "Q?" (id 0) (at 440.69 511.81 90))
+    (property "Reference" "Q15" (id 0) (at 440.69 511.81 90))
     (property "Value" "Q_PMOS_SDG" (id 1) (at 440.69 514.35 90))
     (property "Footprint" "Package_TO_SOT_SMD:TO-252-3_TabPin2" (id 2) (at 438.15 516.89 0)
@@
     )
     (path "/d7e11fd0-e6cc-4f72-bdda-90f2b4e244bb"
-      (reference "#PWR?") (unit 1) (value "GND") (footprint "")
+      (reference "#PWR0176") (unit 1) (value "GND") (footprint "")
     )
     (path "/55cdbc5e-00ae-447d-bee6-68adcd964faf"
@@
     )
     (path "/e2386089-35f2-457e-86e9-aa8c315f254b"
-      (reference "J?") (unit 1) (value "Screw_Terminal_01x02") (footprint "TerminalBlock_Phoenix:TerminalBlock_Phoenix_MKDS-1,5-2-5.08_1x02_P5.08mm_Horizontal")
+      (reference "J22") (unit 1) (value "Screw_Terminal_01x02") (footprint "TerminalBlock_Phoenix:TerminalBlock_Phoenix_MKDS-1,5-2-5.08_1x02_P5.08mm_Horizontal")
     )
     (path "/53df2aa7-9e62-42de-a478-40c5efc9e702"
@@
     )
     (path "/e84e093d-ad9a-46cb-b321-7ca6a57d8ecf"
-      (reference "Q?") (unit 1) (value "Q_PMOS_SDG") (footprint "Package_TO_SOT_SMD:TO-252-3_TabPin2")
+      (reference "Q15") (unit 1) (value "Q_PMOS_SDG") (footprint "Package_TO_SOT_SMD:TO-252-3_TabPin2")
     )
     (path "/90d43173-1036-4d37-973c-c7de805848b2"
@@
     )
     (path "/3bfc8bde-ee7b-4445-92dc-541dd15c34b5"
-      (reference "R?") (unit 1) (value "10K") (footprint "Resistor_SMD:R_1206_3216Metric_Pad1.30x1.75mm_HandSolder")
+      (reference "R46") (unit 1) (value "10K") (footprint "Resistor_SMD:R_1206_3216Metric_Pad1.30x1.75mm_HandSolder")
     )
     (path "/f1f7d6db-21ee-4f0d-910d-6768acba8f9c"
