File: Hardware/LED Strip Controller/Server Rack LED Controller.kicad_sch (KiCad schematic)
At the start: 172 parts, among them J1 LED_ONE_PWR, J10 UART, J11 CONN_2, J12 LED_THREE_PWR, J13 CONN_3, J14 LED_FOUR_PWR, J15 Conn_01x06_Male, J16 CONN_4, J17 TST, J18 Conn_01x02_Female, J19 Conn_02x04_Odd_Even, J2 Screw_Terminal_01x02, J20 Conn_02x04_Odd_Even, J21 Conn_01x02_Female, J22 Screw_Terminal_01x02, J3 PWR_SWITCH, J4 Conn_02x03_Odd_Even, J5 Conn_01x03_Female, J6 CONN_1, J7 LED_TWO_PWR, J8 SWD, J9 USB_B_Micro, Q1 IRF510N, Q10 IRF510N, Q11 IRF510N, Q12 IRF510N, Q13 IRF510N, Q14 IRF510N, Q15 Q_PMOS_SDG, Q2 IRF510N, Q3 Q_PMOS_SDG, Q4 IRF510N, Q5 IRF510N, Q6 IRF510N, Q7 IRF510N, Q8 IRF510N, Q9 IRF510N, SW1 SW_Push_Dual, U1 STM32F103C8Tx, U2 LM2596S-5, U3 LD1117S50TR_SOT223, U4 LD39050PU33R, U5 INA169, U6 USBLC6-2SC6, Y1 Crystal, Y2 8MHz

Commit message: Adding documentation regarding C# User Interface design
Parts:
- U4: footprint DFN-6-1EP_3x3mm_P0.95mm_EP1.7x2.6mm -> Package_DFN_QFN:DFN-6-1EP_3x3mm_P0.95mm_EP1.7x2.6mm
Changed lines of the file:
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@@
     (property "Reference" "U4" (id 0) (at 422.91 208.28 0))
     (property "Value" "LD39050PU33R" (id 1) (at 422.91 210.82 0))
-    (property "Footprint" "DFN-6-1EP_3x3mm_P0.95mm_EP1.7x2.6mm" (id 2) (at 422.91 220.98 0)
+    (property "Footprint" "Package_DFN_QFN:DFN-6-1EP_3x3mm_P0.95mm_EP1.7x2.6mm" (id 2) (at 422.91 220.98 0)
       (effects (font (size 1.27 1.27)) (justify left bottom) hide)
     )
@@
     )
     (path "/a89c8c89-6fe9-4f85-a45b-1aa4a735e99c"
-      (reference "U4") (unit 1) (value "LD39050PU33R") (footprint "DFN-6-1EP_3x3mm_P0.95mm_EP1.7x2.6mm")
+      (reference "U4") (unit 1) (value "LD39050PU33R") (footprint "Package_DFN_QFN:DFN-6-1EP_3x3mm_P0.95mm_EP1.7x2.6mm")
     )
     (path "/2fad9d0d-4f9c-4cc3-8f84-502a9f8d46d3"
